File: PCB/cap_ref_v1.0.brd (EAGLE design)
At the start: 60 x 60 mm, 1 part

Commit message: final_version of v1.0 HW
Parts:
- removed U$1: CAPRES_PADS, connectors:CAPRES_PADS
Connections:
- removed net S00: U$1.P7
- removed net S01: U$1.P6
- removed net S02: U$1.P5
- removed net S03: U$1.P4
- removed net S04: U$1.P3
- removed net S05: U$1.P2
- removed net S06: U$1.P1
- removed net S07: U$1.P0
Routing:
- net S04: track 55.0 -> 0.00 mm, vias 1 -> 0
- net S03: track 54.9 -> 0.00 mm, vias 1 -> 0
- net S05: track 46.1 -> 0.00 mm, vias 1 -> 0
- net S02: track 43.3 -> 0.00 mm, vias 1 -> 0
- net S06: track 28.6 -> 0.00 mm, vias 1 -> 0
- net S01: track 28.0 -> 0.00 mm, vias 1 -> 0
- net S07: track 10.3 -> 0.00 mm, vias 1 -> 0
- net S00: track 10.2 -> 0.00 mm, vias 1 -> 0
- removed copper zone on layer 16, net RX
- removed copper zone on layer 1, net S00
- removed copper zone on layer 1, net S01
- removed copper zone on layer 1, net S02
- removed copper zone on layer 1, net S03
- removed copper zone on layer 1, net S04
- removed copper zone on layer 1, net S05
- removed copper zone on layer 1, net S06
- removed copper zone on layer 1, net S07
Other:
- board size 60 x 60 mm -> 70 x 70 mm
