File: PCB/cap_mother_v1.0.sch (EAGLE design)
At the start: 33 parts, among them IC1 STM32L431KBU6TR, IC2 ADG701LBRJZ-REEL7, IC3 AD8605ARTZ-REEL7, IC4 AD8605ARTZ-REEL7, IC5 74HC164PW,118, U4 MIC5501-3.0YM5-TR

Commit message: final_version of v1.0 HW
Parts:
- removed C11: 100n, rcl:C-EUC0603
- removed R5, R6: 100k, rcl:R-EU_R0603
- added D1: SMDA05-6.TBT, SamacSys_Parts:SMDA05-6.TBT
- added IC6: MCP40D18T-103E_LT, SamacSys_Parts:MCP40D18T-103E_LT
- added J1: 10114828-11108LF, SamacSys_Parts:10114828-11108LF
- added R1: 0R, rcl:R-EU_R0603
Connections:
- removed net T_EN: IC1.PA9, IC5.DSB
- removed net T_RST: IC1.PA10, IC5.!MR
- new net N$1: IC4.+IN, R1.1
- new net SCL: IC1.PB6, IC6.SCL
- new net SDA: IC1.PB7, IC6.SDA
- net +3V3: now also IC5.!MR, IC5.DSB, IC6.VDD; no longer C11.2
- net BIAS_IN: now also R1.2; no longer IC4.+IN
- net CAN1_RX: now also D1.K3, J1.4
- net CAN1_TX: now also D1.K4, J1.5
- net GND: now also D1.A1, D1.A2, IC6.VSS, J1.8, J1.MP1, J1.MP2; no longer C11.1, R6.2
- net IN-: now also IC6.W; no longer R5.1, R6.1
- net OUT_: now also IC6.A; no longer R5.2
- net USART1_RX: now also D1.K6, IC1.PA10, J1.2; no longer IC1.PB7
- net USART1_TX: now also D1.K5, IC1.PA9, J1.3; no longer IC1.PB6
- net VDD: now also D1.K1, J1.1

Commit message: fw hw setup
Changed lines of the file:
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@@
 <pinref part="C20" gate="G$1" pin="1"/>
 <pinref part="GND7" gate="1" pin="GND"/>
-<wire x1="-78.74" y1="123.19" x2="-78.74" y2="119.38" width="0.1524" layer="91"/>
+<wire x1="-78.74" y1="123.19" x2="-78.74" y2="120.65" width="0.1524" layer="91"/>
+<wire x1="-78.74" y1="120.65" x2="-78.74" y2="119.38" width="0.1524" layer="91"/>
+<wire x1="-74.93" y1="120.65" x2="-78.74" y2="120.65" width="0.1524" layer="91"/>
+<junction x="-78.74" y="120.65"/>
 </segment>
 <segment>
